File: Hardware/Buck_Regulator_AP3429A_1V8/Buck_Regulator_AP3429A_1V8.brd (EAGLE design)
At the start: 25.4 x 25.4 mm, 53 parts, among them J1 Screw Terminal, J2 POWER_JACKPOWER_JACK_SLOT_COM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, J3 Breakout Headers, U1 AP3429/A

Commit message: Updated panelized files
Adjusted via to no longer be in the way of the bStop on the back for the thermal pad on the backside. Included ordering instructions on the brd files for both 1.8V and 3.3V
Parts:
- added U$17: (no value), SparkFun-Aesthetics:ORDERING_INSTRUCTIONS
Routing:
- net N$3: track 36.4 -> 37.5 mm
Other:
- board text added: "Board thickness is 1.6mm 2-Layer 1oz copper outer 1oz copper inner"
Changed lines of the file:
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@@
 <layer number="44" name="Drills" color="7" fill="1" visible="no" active="yes"/>
 <layer number="45" name="Holes" color="7" fill="1" visible="yes" active="yes"/>
-<layer number="46" name="Milling" color="3" fill="1" visible="no" active="yes"/>
+<layer number="46" name="Milling" color="3" fill="1" visible="yes" active="yes"/>
 <layer number="47" name="Measures" color="7" fill="1" visible="no" active="yes"/>
 <layer number="48" name="Document" color="7" fill="1" visible="no" active="yes"/>
@@
 <dimension x1="24.13" y1="7.62" x2="0" y2="7.62" x3="12.065" y3="-21.59" textsize="1.778" textratio="15" layer="47" unit="inch"/>
 <dimension x1="0" y1="0" x2="25.4" y2="0" x3="12.7" y3="-26.67" textsize="1.778" textratio="15" layer="47" unit="inch"/>
+<text x="33.528" y="4.699" size="1.778" layer="51" font="vector">Board thickness is 1.6mm
+2-Layer
+1oz copper outer
+1oz copper inner</text>
 </plain>
 <attributes>
@@
 </element>
 <element name="J2" library="SparkFun-Connectors" package="POWER_JACK_PTH_SLOT_BOTH" value="POWER_JACKPOWER_JACK_SLOT_COMBO" x="13.335" y="24.003" smashed="yes" rot="R90"/>
+<element name="U$17" library="SparkFun-Aesthetics" package="ORDERING_INSTRUCTIONS" value="" x="31.75" y="25.4" smashed="yes"/>
 </elements>
 <signals>
@@
 <wire x1="4.9657" y1="20.9677" x2="4.572" y2="20.574" width="0.2032" layer="16"/>
 <wire x1="4.572" y1="20.574" x2="1.905" y2="20.574" width="0.2032" layer="16"/>
-<wire x1="13.247" y1="2.667" x2="17.184" y2="2.667" width="0.2032" layer="1"/>
-<wire x1="13.247" y1="2.667" x2="12.612" y2="3.302" width="0.2032" layer="1"/>
-<wire x1="12.612" y1="3.302" x2="7.493" y2="3.302" width="0.2032" layer="1"/>
-<via x="6.477" y="4.318" extent="1-16" drill="0.381"/>
-<wire x1="6.477" y1="4.318" x2="7.493" y2="3.302" width="0.2032" layer="1"/>
 <wire x1="0.762" y1="19.431" x2="0.762" y2="7.366" width="0.2032" layer="16"/>
 <wire x1="0.762" y1="7.366" x2="2.54" y2="5.588" width="0.2032" layer="16"/>
-<wire x1="5.207" y1="5.588" x2="6.477" y2="4.318" width="0.2032" layer="16"/>
-<wire x1="5.207" y1="5.588" x2="2.54" y2="5.588" width="0.2032" layer="16"/>
+<via x="15.44930625" y="2.667" extent="1-16" drill="0.35"/>
+<wire x1="15.44930625" y1="2.667" x2="17.184" y2="2.667" width="0.2032" layer="1"/>
+<wire x1="5.207" y1="5.588" x2="5.588" y2="5.207" width="0.2032" layer="16"/>
+<wire x1="2.54" y1="5.588" x2="5.207" y2="5.588" width="0.2032" layer="16"/>
+<wire x1="5.588" y1="5.207" x2="5.588" y2="3.302" width="0.2032" layer="16"/>
+<wire x1="5.588" y1="3.302" x2="6.223" y2="2.667" width="0.2032" layer="16"/>
+<wire x1="6.223" y1="2.667" x2="15.44930625" y2="2.667" width="0.2032" layer="16"/>
 </signal>
 <signal name="N$4">
@@
 <vertex x="19.304" y="5.842"/>
 <vertex x="19.304" y="8.509"/>
-<vertex x="13.97" y="8.509"/>
 <vertex x="13.843" y="8.509"/>
 </polygon>
@@
 </drawing>
 <compatibility>
+<note version="6.3" minversion="6.2.2" severity="warning">
+Since Version 6.2.2 text objects can contain more than one line,
+which will not be processed correctly with this version.
+</note>
 <note version="8.3" severity="warning">
 Since Version 8.3, EAGLE supports URNs for individual library
